File: discrete-receiver/ethernet_interface.kicad_sch (KiCad schematic)
At the start: 15 parts, among them J6 SI-52003-F, U9 LAN8720A

Commit message: :)
Parts:
- C49: Manufacturer Samsung Electro-Mechanics -> (none); Price 0.007USD -> (none)
- C50, C52: Manufacturer Samsung Electro-Mechanics -> (none); Price 0.006USD -> (none)
- C51: Manufacturer FH(Guangdong Fenghua Advanced Tech) -> (none); Price 0.004USD -> (none)
- C53, C54: Manufacturer Samsung Electro-Mechanics -> (none); Price 0.004USD -> (none)
- J6: Availability Unavailable -> (none); Package None -> (none); Price None -> (none)
- R18, R25, R30, R31, R32, R33: Manufacturer UNI-ROYAL(Uniroyal Elec) -> (none); Price 0.004USD -> (none)

Commit message: formatting
Other:
- note added: "TO DO: - Determine if ethernet chip can do 12kΩ instead of 12.1kΩ (Done) - JLC the rest"
- note removed: "TO DO: - Determine if ethernet chip can do 12kΩ instead of 12.1kΩ - JLC the rest"
Changed lines of the file:
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@@
 		)
 	)
-	(text "TO DO:\n- Determine if ethernet chip can do 12kΩ instead of 12.1kΩ\n- JLC the rest"
+	(text "TO DO:\n- Determine if ethernet chip can do 12kΩ instead of 12.1kΩ (Done)\n- JLC the rest"
 		(exclude_from_sim no)
 		(at 49.022 229.87 0)

Commit message: all parts now have footprints
Parts:
- J6: footprint SI-52003-F:BEL_SI-52003-F -> sdr_project:BEL_SI-52003-F
- JP5: footprint (none) -> Jumper:SolderJumper-2_P1.3mm_Open_Pad1.0x1.5mm
Changed lines of the file:
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@@
 		)
 		(instances
-			(project "tayloe_detector"
+			(project "diode_tayloe_sdr"
 				(path "/d18d178d-3f10-4d68-9036-eae71a7d091a/09065ae7-5d3e-4f86-b983-86dca844c240"
 					(reference "#PWR086")
@@
 		)
 		(instances
-			(project "tayloe_detector"
+			(project "diode_tayloe_sdr"
 				(path "/d18d178d-3f10-4d68-9036-eae71a7d091a/09065ae7-5d3e-4f86-b983-86dca844c240"
 					(reference "C50")
@@
 			)
 		)
-		(property "Footprint" ""
+		(property "Footprint" "Jumper:SolderJumper-2_P1.3mm_Open_Pad1.0x1.5mm"
 			(at 83.82 177.8 0)
 			(hide yes)
@@
 		)
 		(instances
-			(project "tayloe_detector"
+			(project "diode_tayloe_sdr"
 				(path "/d18d178d-3f10-4d68-9036-eae71a7d091a/09065ae7-5d3e-4f86-b983-86dca844c240"
 					(reference "JP5")
@@
 		)
 		(instances
-			(project "tayloe_detector"
+			(project "diode_tayloe_sdr"
 				(path "/d18d178d-3f10-4d68-9036-eae71a7d091a/09065ae7-5d3e-4f86-b983-86dca844c240"
 					(reference "#PWR085")
@@
 		)
 		(instances
-			(project "tayloe_detector"
+			(project "diode_tayloe_sdr"
 				(path "/d18d178d-3f10-4d68-9036-eae71a7d091a/09065ae7-5d3e-4f86-b983-86dca844c240"
 					(reference "R31")
@@
 			)
 		)
-		(property "Footprint" "SI-52003-F:BEL_SI-52003-F"
+		(property "Footprint" "sdr_project:BEL_SI-52003-F"
 			(at 101.6 154.94 0)
 			(hide yes)
@@
 		)
 		(instances
-			(project "tayloe_detector"
+			(project "diode_tayloe_sdr"
 				(path "/d18d178d-3f10-4d68-9036-eae71a7d091a/09065ae7-5d3e-4f86-b983-86dca844c240"
 					(reference "J6")
@@
 		)
 		(instances
-			(project "tayloe_detector"
+			(project "diode_tayloe_sdr"
 				(path "/d18d178d-3f10-4d68-9036-eae71a7d091a/09065ae7-5d3e-4f86-b983-86dca844c240"
 					(reference "#PWR076")
@@
 		)
 		(instances
-			(project "tayloe_detector"
+			(project "diode_tayloe_sdr"
 				(path "/d18d178d-3f10-4d68-9036-eae71a7d091a/09065ae7-5d3e-4f86-b983-86dca844c240"
 					(reference "U9")
@@
 		)
 		(instances
-			(project "tayloe_detector"
+			(project "diode_tayloe_sdr"
 				(path "/d18d178d-3f10-4d68-9036-eae71a7d091a/09065ae7-5d3e-4f86-b983-86dca844c240"
 					(reference "R30")
@@
 		)
 		(instances
-			(project "tayloe_detector"
+			(project "diode_tayloe_sdr"
 				(path "/d18d178d-3f10-4d68-9036-eae71a7d091a/09065ae7-5d3e-4f86-b983-86dca844c240"
 					(reference "R32")
@@
 		)
 		(instances
-			(project "tayloe_detector"
+			(project "diode_tayloe_sdr"
 				(path "/d18d178d-3f10-4d68-9036-eae71a7d091a/09065ae7-5d3e-4f86-b983-86dca844c240"
 					(reference "#PWR095")
@@
 		)
 		(instances
-			(project "tayloe_detector"
+			(project "diode_tayloe_sdr"
 				(path "/d18d178d-3f10-4d68-9036-eae71a7d091a/09065ae7-5d3e-4f86-b983-86dca844c240"
 					(reference "#PWR078")
@@
 		)
 		(instances
-			(project "tayloe_detector"
+			(project "diode_tayloe_sdr"
 				(path "/d18d178d-3f10-4d68-9036-eae71a7d091a/09065ae7-5d3e-4f86-b983-86dca844c240"
 					(reference "#PWR084")
@@
 		)
 		(instances
-			(project "tayloe_detector"
+			(project "diode_tayloe_sdr"
 				(path "/d18d178d-3f10-4d68-9036-eae71a7d091a/09065ae7-5d3e-4f86-b983-86dca844c240"
 					(reference "C53")
@@
 		)
 		(instances
-			(project "tayloe_detector"
+			(project "diode_tayloe_sdr"
 				(path "/d18d178d-3f10-4d68-9036-eae71a7d091a/09065ae7-5d3e-4f86-b983-86dca844c240"
 					(reference "#PWR083")
@@
 		)
 		(instances
-			(project "tayloe_detector"
+			(project "diode_tayloe_sdr"
 				(path "/d18d178d-3f10-4d68-9036-eae71a7d091a/09065ae7-5d3e-4f86-b983-86dca844c240"
 					(reference "#PWR079")
@@
 		)
 		(instances
-			(project "tayloe_detector"
+			(project "diode_tayloe_sdr"
 				(path "/d18d178d-3f10-4d68-9036-eae71a7d091a/09065ae7-5d3e-4f86-b983-86dca844c240"
 					(reference "#PWR077")
@@
 		)
 		(instances
-			(project "tayloe_detector"
+			(project "diode_tayloe_sdr"
 				(path "/d18d178d-3f10-4d68-9036-eae71a7d091a/09065ae7-5d3e-4f86-b983-86dca844c240"
 					(reference "R18")
@@
 		)
 		(instances
-			(project "tayloe_detector"
+			(project "diode_tayloe_sdr"
 				(path "/d18d178d-3f10-4d68-9036-eae71a7d091a/09065ae7-5d3e-4f86-b983-86dca844c240"
 					(reference "R25")
@@
 		)
 		(instances
-			(project "tayloe_detector"
+			(project "diode_tayloe_sdr"
 				(path "/d18d178d-3f10-4d68-9036-eae71a7d091a/09065ae7-5d3e-4f86-b983-86dca844c240"
 					(reference "C52")
@@
 		)
 		(instances
-			(project "tayloe_detector"
+			(project "diode_tayloe_sdr"
 				(path "/d18d178d-3f10-4d68-9036-eae71a7d091a/09065ae7-5d3e-4f86-b983-86dca844c240"
 					(reference "C54")
@@
 		)
 		(instances
-			(project "tayloe_detector"
+			(project "diode_tayloe_sdr"
 				(path "/d18d178d-3f10-4d68-9036-eae71a7d091a/09065ae7-5d3e-4f86-b983-86dca844c240"
 					(reference "R33")
@@
 		)
 		(instances
-			(project "tayloe_detector"
+			(project "diode_tayloe_sdr"
 				(path "/d18d178d-3f10-4d68-9036-eae71a7d091a/09065ae7-5d3e-4f86-b983-86dca844c240"
 					(reference "#PWR050")
@@
 		)
 		(instances
-			(project "tayloe_detector"
+			(project "diode_tayloe_sdr"
 				(path "/d18d178d-3f10-4d68-9036-eae71a7d091a/09065ae7-5d3e-4f86-b983-86dca844c240"
 					(reference "C49")
@@
 		)
 		(instances
-			(project "tayloe_detector"
+			(project "diode_tayloe_sdr"
 				(path "/d18d178d-3f10-4d68-9036-eae71a7d091a/09065ae7-5d3e-4f86-b983-86dca844c240"
 					(reference "C51")

Commit message: PCB Updates
Parts:
- added R36: 100Ω, PCM_JLCPCB:R_0402, symbol PCM_JLCPCB-Resistors:0402,100Ω
Connections:
- net at U9.24 (RBIAS): now also R36.1; no longer R18.1
- new net: R18.1, R36.2
Other:
- moved on the sheet: R18

Commit message: Improved silkscreen and added 3D models to PCB
Made font size of components smaller to improve clarity as to what label is associated with what component.

Also, added 3D models for components that did not have any, and also assigned 3D models for components that we had models for but had forgotten to assign them.
Parts:
- J6: LCSC (none) -> C6488114; MF Stewart Connector -> (none); MP SI-52003-F -> (none)
Changed lines of the file:
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@@
 			)
 		)
-		(property "MF" "Stewart Connector"
+		(property "LCSC" "C6488114"
 			(at 101.6 154.94 0)
 			(hide yes)
@@
 					(size 1.27 1.27)
 				)
-				(justify bottom)
 			)
 		)
-		(property "MP" "SI-52003-F"
-			(at 101.6 154.94 0)
-			(hide yes)
-			(show_name no)
-			(do_not_autoplace no)
-			(effects
-				(font
-					(size 1.27 1.27)
-				)
-				(justify bottom)
-			)
-		)
