File: discrete-receiver/diode_tayloe_sdr.kicad_sch (KiCad schematic)
At the start: 17 parts, among them J5 Display Connector, X1 YC24.576MUBCE2O

Commit message: PCB Updates
Other:
- sheet ADC ports: added ~{ADC_RST}; removed none
- sheet Pico ports: added ~{ADC_RST}; removed none
Changed lines of the file:
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@@
 	)
 	(junction
-		(at 45.72 53.34)
+		(at 55.88 39.37)
 		(diameter 0)
 		(color 0 0 0 0)
 	)
 	(junction
-		(at 55.88 39.37)
+		(at 33.02 72.39)
 		(diameter 0)
 		(color 0 0 0 0)
 	)
 	(junction
-		(at 33.02 72.39)
+		(at 45.72 48.26)
 		(diameter 0)
 		(color 0 0 0 0)
@@
 	)
 	(junction
-		(at 45.72 48.26)
+		(at 45.72 53.34)
 		(diameter 0)
 		(color 0 0 0 0)
@@
 	(wire
 		(pts
+			(xy 123.19 146.05) (xy 123.19 109.22)
+		)
+		(stroke
+			(width 0)
+			(type default)
+		)
+	)
+	(wire
+		(pts
 			(xy 128.27 140.97) (xy 142.24 140.97)
 		)
@@
 	(wire
 		(pts
+			(xy 142.24 146.05) (xy 123.19 146.05)
+		)
+		(stroke
+			(width 0)
+			(type default)
+		)
+	)
+	(wire
+		(pts
 			(xy 185.42 130.81) (xy 190.5 130.81)
 		)
@@
 	(wire
 		(pts
+			(xy 123.19 109.22) (xy 120.65 109.22)
+		)
+		(stroke
+			(width 0)
+			(type default)
+		)
+	)
+	(wire
+		(pts
 			(xy 45.72 48.26) (xy 83.82 48.26)
 		)
@@
 	(sheet
 		(at 83.82 42.418)
-		(size 36.83 65.786)
+		(size 36.83 70.612)
 		(exclude_from_sim no)
 		(in_bom yes)
@@
 		)
 		(property "Sheetfile" "pico.kicad_sch"
-			(at 83.82 108.7886 0)
+			(at 83.82 113.6146 0)
 			(show_name no)
 			(do_not_autoplace no)
@@
 			)
 		)
+		(pin "~{ADC_RST}" input
+			(at 120.65 109.22 0)
+			(effects
+				(font
+					(size 1.27 1.27)
+				)
+				(justify right)
+			)
+		)
 		(instances
 			(project "diode_tayloe_sdr"
@@
 	(sheet
 		(at 142.24 128.016)
-		(size 31.75 19.304)
+		(size 31.75 21.844)
 		(exclude_from_sim no)
 		(in_bom yes)
@@
 		)
 		(property "Sheetfile" "adc.kicad_sch"
-			(at 142.24 147.9046 0)
+			(at 142.24 150.4446 0)
 			(show_name no)
 			(do_not_autoplace no)
@@
 			(effects
 				(font
+					(size 1.27 1.27)
+				)
+				(justify left)
+			)
+		)
+		(pin "~{ADC_RST}" input
+			(at 142.24 146.05 180)
+			(effects
+				(font
